File: rambo/rambo.kicad_pcb (KiCad board)
At the start: 2 copper layers, 130.9 x 81.3 mm, 43 parts, among them J1 Barrel_Jack_Switch, J2 USB_B, J3 Conn_02x25_Odd_Even, Q1 2N7000, SW1 SW_DIP_x04, U1 74LS139, U10 74HCT04, U11 74LS245, U12 74HCT00, U13 74LS85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

Commit message: inverted select fix
Connections:
- U10 pad 8: unconnected-(U10-Pad8) -> Net-(U10-Pad8)
- U10 pad 9: unconnected-(U10-Pad9) -> Net-(U12-Pad2)
- U11 pad 19: Net-(U11-Pad19) -> Net-(U10-Pad8)
- U12 pad 2: Net-(U11-Pad19) -> Net-(U12-Pad2)
- U12 pad 5: Net-(U11-Pad19) -> Net-(U12-Pad2)
- U13 pad 6: Net-(U11-Pad19) -> Net-(U12-Pad2)
Routing:
- net Net-(U11-Pad19): track 84.0 -> 0.00 mm, vias 1 -> 0
- net Net-(U10-Pad8): track 0.00 -> 66.0 mm, vias 0 -> 1
- net Net-(U12-Pad2): track 0.00 -> 44.1 mm
Other:
- board text added: "TRS-80 Model 3 high speed RAM board Rev. B"
- board text removed: "TRS-80 Model 3 high speed RAM board"
